File: fc_rocket.sch (EAGLE design)
At the start: 31 parts, among them IC1 7805TV, J1 1X2-3.5MM, J2 1X2-3.5MM, J3 1X2-3.5MM, J4 1X2-3.5MM, J5 1X2-3.5MM, J6 1X2-3.5MM, U2 GY-521MPU6050

Commit message: finised auto router
Parts:
- removed J1: 1X2-3.5MM, adafruit:1X2-3.5MM
- added S1: (no value), adafruit:EG1218S
Connections:
- removed net BATT+: J1.2, J2.2
- new net VIN: ARDUINO_NANO1.VIN, S1.S
- net 12V: now also J2.2; no longer J2.1
- net 5V: now also S1.P
- net GND: now also ARDUINO_NANO1.GND@2, J2.1; no longer J1.1
Other:
- moved on the sheet: ARDUINO_NANO1, C2, C3, C4, D1, IC1, LS2, Q1, Q2, Q3, Q4, Q5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

Commit message: backup
Parts:
- R3: value 40ohm -> 4.7k; device adafruit:FLIPFLOP-RES -> SparkFun-Resistors:4.7KOHM-0603-1/10W-1%
Changed lines of the file:
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@@
 <part name="GND1" library="supply1" library_urn="urn:adsk.eagle:library:371" deviceset="GND" device=""/>
 <part name="SUPPLY1" library="SparkFun-PowerSymbols" library_urn="urn:adsk.eagle:library:530" deviceset="5V" device=""/>
-<part name="R3" library="adafruit" deviceset="FLIPFLOP-RES" device="" value="40ohm"/>
+<part name="R3" library="SparkFun-Resistors" library_urn="urn:adsk.eagle:library:532" deviceset="4.7KOHM" device="-0603-1/10W-1%" package3d_urn="urn:adsk.eagle:package:39650/1" value="4.7k"/>
 <part name="R4" library="adafruit" deviceset="FLIPFLOP-RES" device="" value="1ohm"/>
 <part name="R5" library="adafruit" deviceset="FLIPFLOP-RES" device="" value="1ohm"/>
